Commit message: joint4 upper limit 145 deg (WLKATA's own URDF), was 179 deg
Compared with github.com/wlkata/Wlkata_Mirobot_Ros2 (2026-10-28): all other limits of
mirobot_urdf_2.urdf (the one MoveIt loads) are within WLKATA's; joint4 upper was 179.3 deg vs
their 145 deg. To be confirmed against the Mirobot manual / firmware soft limits.

Co-Authored-By: Claude Opus 5.5 <noreply@anthropic.com>
Claude-Session: https://claude.ai/code/session_01W7jf3rwZQovCLP6XtyJ8V1

File: src/mirobot_description/urdf/mirobot_urdf_2.urdf (robot description, URDF)
Before this commit: robot mirobot, 9 links, 8 joints
Joints:
- joint joint4: limit lower=-3.13 upper=3.13 effort=200 velocity=200 -> lower=-3.13 upper=2.53 effort=200 velocity=200
